Commit message: Update ugv.urdf.xacro

File: quadrotors_landing_vision/models/husky/urdf/ugv.urdf.xacro (robot description, xacro)
@@ -1,16 +1,3 @@
 <?xml version="1.0"?>
-<!--
-  This file is part of the uav_landing_sim distribution (https://github.com/dimianx/uav_landing_sim).
-  Copyright (c) 2025 Dmitry Anikin.
-  This program is free software: you can redistribute it and/or modify
-  it under the terms of the GNU General Public License as published by
-  the Free Software Foundation, version 3.
-  This program is distributed in the hope that it will be useful, but
-  WITHOUT ANY WARRANTY; without even the implied warranty of
-  MERCHANTABILITY or FITNESS FOR A PARTICULAR PURPOSE. See the GNU
-  General Public License for more details.
-  You should have received a copy of the GNU General Public License
-  along with this program. If not, see <http://www.gnu.org/licenses/>.
--->
 <robot name="husky" xmlns:xacro="http://ros.org/wiki/xacro">
   <xacro:include filename="$(find husky_description)/urdf/husky.urdf.xacro" />
@@ -19,10 +6,10 @@
       <cast_shadows>true</cast_shadows>
       <geometry>
-        <mesh filename="package://uav_landing_sim/models/husky/meshes/platform.dae" scale="0.5 0.5 0.5"/>
+        <mesh filename="package://quadrotors_landing_vision/models/husky/meshes/platform.dae" scale="0.5 0.5 0.5"/>
       </geometry>
     </visual>
     <collision>
       <geometry>
-        <mesh filename="package://uav_landing_sim/models/husky/meshes/platform.dae" scale="0.5 0.5 0.5"/>
+        <mesh filename="package://quadrotors_landing_vision/models/husky/meshes/platform.dae" scale="0.5 0.5 0.5"/>
       </geometry>
     </collision>
@@ -37,10 +24,10 @@
       <cast_shadows>true</cast_shadows>
       <geometry>
-        <mesh filename="package://uav_landing_sim/models/husky/meshes/uwb_anchor.dae" scale="1 1 1"/>
+        <mesh filename="package://quadrotors_landing_vision/models/husky/meshes/uwb_anchor.dae" scale="1 1 1"/>
       </geometry>
     </visual>
     <collision>
       <geometry>
-        <mesh filename="package://uav_landing_sim/models/husky/meshes/uwb_anchor.dae" scale="1 1 1"/>
+        <mesh filename="package://quadrotors_landing_vision/models/husky/meshes/uwb_anchor.dae" scale="1 1 1"/>
       </geometry>
     </collision>
@@ -55,10 +42,10 @@
       <cast_shadows>true</cast_shadows>
       <geometry>
-        <mesh filename="package://uav_landing_sim/models/husky/meshes/uwb_anchor.dae" scale="1 1 1"/>
+        <mesh filename="package://quadrotors_landing_vision/models/husky/meshes/uwb_anchor.dae" scale="1 1 1"/>
       </geometry>
     </visual>
     <collision>
       <geometry>
-        <mesh filename="package://uav_landing_sim/models/husky/meshes/uwb_anchor.dae" scale="1 1 1"/>
+        <mesh filename="package://quadrotors_landing_vision/models/husky/meshes/uwb_anchor.dae" scale="1 1 1"/>
       </geometry>
     </collision>
@@ -73,10 +60,10 @@
       <cast_shadows>true</cast_shadows>
       <geometry>
-        <mesh filename="package://uav_landing_sim/models/husky/meshes/uwb_anchor.dae" scale="1 1 1"/>
+        <mesh filename="package://quadrotors_landing_vision/models/husky/meshes/uwb_anchor.dae" scale="1 1 1"/>
       </geometry>
     </visual>
     <collision>
       <geometry>
-        <mesh filename="package://uav_landing_sim/models/husky/meshes/uwb_anchor.dae" scale="1 1 1"/>
+        <mesh filename="package://quadrotors_landing_vision/models/husky/meshes/uwb_anchor.dae" scale="1 1 1"/>
       </geometry>
     </collision>
@@ -91,10 +78,10 @@
       <cast_shadows>true</cast_shadows>
       <geometry>
-        <mesh filename="package://uav_landing_sim/models/husky/meshes/uwb_anchor.dae" scale="1 1 1"/>
+        <mesh filename="package://quadrotors_landing_vision/models/husky/meshes/uwb_anchor.dae" scale="1 1 1"/>
       </geometry>
     </visual>
     <collision>
       <geometry>
-        <mesh filename="package://uav_landing_sim/models/husky/meshes/uwb_anchor.dae" scale="1 1 1"/>
+        <mesh filename="package://quadrotors_landing_vision/models/husky/meshes/uwb_anchor.dae" scale="1 1 1"/>
       </geometry>
     </collision>
@@ -109,10 +96,10 @@
       <cast_shadows>true</cast_shadows>
       <geometry>
-        <mesh filename="package://uav_landing_sim/models/husky/meshes/marker.dae" />
+        <mesh filename="package://quadrotors_landing_vision/models/husky/meshes/marker.dae" />
       </geometry>
     </visual>
     <collision>
       <geometry>
-        <mesh filename="package://uav_landing_sim/models/husky/meshes/marker.dae" />
+        <mesh filename="package://quadrotors_landing_vision/models/husky/meshes/marker.dae" />
       </geometry>
     </collision>
@@ -127,10 +114,10 @@
       <cast_shadows>true</cast_shadows>
       <geometry>
-        <mesh filename="package://uav_landing_sim/models/husky/meshes/diode.dae" scale="0.4 0.4 0.4"/>
+        <mesh filename="package://quadrotors_landing_vision/models/husky/meshes/diode.dae" scale="0.4 0.4 0.4"/>
       </geometry>
     </visual>
     <collision>
       <geometry>
-        <mesh filename="package://uav_landing_sim/models/husky/meshes/diode.dae" scale="0.4 0.4 0.4"/>
+        <mesh filename="package://quadrotors_landing_vision/models/husky/meshes/diode.dae" scale="0.4 0.4 0.4"/>
       </geometry>
     </collision>
@@ -145,10 +132,10 @@
       <cast_shadows>true</cast_shadows>
       <geometry>
-        <mesh filename="package://uav_landing_sim/models/husky/meshes/diode.dae" scale="0.4 0.4 0.4"/>
+        <mesh filename="package://quadrotors_landing_vision/models/husky/meshes/diode.dae" scale="0.4 0.4 0.4"/>
       </geometry>
     </visual>
     <collision>
       <geometry>
-        <mesh filename="package://uav_landing_sim/models/husky/meshes/diode.dae" scale="0.4 0.4 0.4"/>
+        <mesh filename="package://quadrotors_landing_vision/models/husky/meshes/diode.dae" scale="0.4 0.4 0.4"/>
       </geometry>
     </collision>
@@ -163,10 +150,10 @@
       <cast_shadows>true</cast_shadows>
       <geometry>
-        <mesh filename="package://uav_landing_sim/models/husky/meshes/diode.dae" scale="0.4 0.4 0.4"/>
+        <mesh filename="package://quadrotors_landing_vision/models/husky/meshes/diode.dae" scale="0.4 0.4 0.4"/>
       </geometry>
     </visual>
     <collision>
       <geometry>
-        <mesh filename="package://uav_landing_sim/models/husky/meshes/diode.dae" scale="0.4 0.4 0.4"/>
+        <mesh filename="package://quadrotors_landing_vision/models/husky/meshes/diode.dae" scale="0.4 0.4 0.4"/>
       </geometry>
     </collision>
@@ -181,10 +168,10 @@
       <cast_shadows>true</cast_shadows>
       <geometry>
-        <mesh filename="package://uav_landing_sim/models/husky/meshes/diode.dae" scale="0.4 0.4 0.4"/>
+        <mesh filename="package://quadrotors_landing_vision/models/husky/meshes/diode.dae" scale="0.4 0.4 0.4"/>
       </geometry>
     </visual>
     <collision>
       <geometry>
-        <mesh filename="package://uav_landing_sim/models/husky/meshes/diode.dae" scale="0.4 0.4 0.4"/>
+        <mesh filename="package://quadrotors_landing_vision/models/husky/meshes/diode.dae" scale="0.4 0.4 0.4"/>
       </geometry>
     </collision>
